File: pure_spindel_pwm/main.sch (EAGLE design)
At the start: 8 parts, among them J1 SPINDEL, J2 POWER, J3 CONTROL, Q1 IRF530, U1 IR2117SO8-2

Commit message: pure_spindel_pwm: fix: invalid capacitor nets
Connections:
- removed net N$1: C1.1, D1.C
- net GND_48V: now also C1.2
- net VB: now also C1.1, D1.C; no longer C1.2
Changed lines of the file:
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@@
 </busses>
 <nets>
-<net name="VB" class="0">
-<segment>
-<pinref part="U1" gate="U1" pin="VB"/>
-<pinref part="C1" gate="G$1" pin="2"/>
-<wire x1="88.9" y1="60.96" x2="93.98" y2="60.96" width="0.1524" layer="91"/>
-<wire x1="93.98" y1="60.96" x2="93.98" y2="63.5" width="0.1524" layer="91"/>
-</segment>
-</net>
-<net name="N$1" class="0">
-<segment>
-<pinref part="C1" gate="G$1" pin="1"/>
-<pinref part="D1" gate="G$1" pin="C"/>
-<wire x1="93.98" y1="71.12" x2="93.98" y2="73.66" width="0.1524" layer="91"/>
-<wire x1="93.98" y1="73.66" x2="78.74" y2="73.66" width="0.1524" layer="91"/>
-</segment>
-</net>
 <net name="GATE" class="0">
 <segment>
@@
 <wire x1="101.6" y1="53.34" x2="101.6" y2="50.8" width="0.1524" layer="91"/>
 <pinref part="U1" gate="U1" pin="VS"/>
-<wire x1="88.9" y1="50.8" x2="101.6" y2="50.8" width="0.1524" layer="91"/>
+<wire x1="88.9" y1="50.8" x2="93.98" y2="50.8" width="0.1524" layer="91"/>
 <pinref part="J2" gate="G$1" pin="1"/>
+<wire x1="93.98" y1="50.8" x2="101.6" y2="50.8" width="0.1524" layer="91"/>
 <wire x1="101.6" y1="50.8" x2="101.6" y2="35.56" width="0.1524" layer="91"/>
 <junction x="101.6" y="50.8"/>
+<pinref part="C1" gate="G$1" pin="2"/>
+<wire x1="93.98" y1="63.5" x2="93.98" y2="50.8" width="0.1524" layer="91"/>
+<junction x="93.98" y="50.8"/>
 </segment>
 </net>
@@
 </segment>
 </net>
+<net name="VB" class="0">
+<segment>
+<pinref part="U1" gate="U1" pin="VB"/>
+<wire x1="88.9" y1="60.96" x2="88.9" y2="73.66" width="0.1524" layer="91"/>
+<pinref part="D1" gate="G$1" pin="C"/>
+<wire x1="88.9" y1="73.66" x2="78.74" y2="73.66" width="0.1524" layer="91"/>
+<pinref part="C1" gate="G$1" pin="1"/>
+<wire x1="93.98" y1="71.12" x2="93.98" y2="73.66" width="0.1524" layer="91"/>
+<wire x1="93.98" y1="73.66" x2="88.9" y2="73.66" width="0.1524" layer="91"/>
+<junction x="88.9" y="73.66"/>
+</segment>
+</net>
